Commit message: Updated CMakeLists.txt, package.xml, and README.md + launch file for RViz now works + minor changes

File: xacro/plane_with_restitution.urdf.xacro (robot description, xacro)
@@ -1,29 +1,29 @@
 <?xml version="1.0" ?>
 <robot name="plane">
-  <link name="planeLink">
-  <contact>
-      <lateral_friction value="1.0"/>
-      <restitution value="0.0"/>
-  </contact>
-    <inertial>
-      <origin rpy="0 0 0" xyz="0 0 0"/>
-       <mass value=".0"/>
-       <inertia ixx="0" ixy="0" ixz="0" iyy="0" iyz="0" izz="0"/>
-    </inertial>
-    <visual>
-      <origin rpy="0 0 0" xyz="0 0 0"/>
-      <geometry>
-      <mesh filename="file://$(find solo_description)/meshes/plane.obj" scale="1 1 1"/>
-      </geometry>
-       <material name="white">
-        <color rgba="1 1 1 1"/>
-      </material>
-    </visual>
-    <collision>
-      <origin rpy="0 0 0" xyz="0 0 -5"/>
-      <geometry>
-      <box size="30 30 10"/>
-      </geometry>
-    </collision>
-  </link>
+    <link name="planeLink">
+    <contact>
+        <lateral_friction value="1.0"/>
+        <restitution value="0.0"/>
+    </contact>
+        <inertial>
+            <origin rpy="0 0 0" xyz="0 0 0"/>
+            <mass value=".0"/>
+            <inertia ixx="0" ixy="0" ixz="0" iyy="0" iyz="0" izz="0"/>
+        </inertial>
+        <visual>
+            <origin rpy="0 0 0" xyz="0 0 0"/>
+            <geometry>
+                <mesh filename="file://$(find solo_description)/meshes/plane.obj" scale="1 1 1"/>
+            </geometry>
+            <material name="white">
+                <color rgba="1 1 1 1"/>
+            </material>
+        </visual>
+        <collision>
+            <origin rpy="0 0 0" xyz="0 0 -5"/>
+            <geometry>
+                <box size="30 30 10"/>
+            </geometry>
+        </collision>
+    </link>
 </robot>

File: xacro/solo12.urdf.xacro (robot description, xacro)
@@ -1,93 +1,93 @@
 <?xml version="1.0" ?>
 <robot name="solo"
-  xmlns:controller="http://playerstage.sourceforge.net/gazebo/xmlschema/#controller"
-  xmlns:interface="http://playerstage.sourceforge.net/gazebo/xmlschema/#interface"
-  xmlns:sensor="http://playerstage.sourceforge.net/gazebo/xmlschema/#sensor"
-  xmlns:xacro="http://playerstage.sourceforge.net/gazebo/xmlschema/#interface">
-  <xacro:property name="color_name" value="grey" />
-  <xacro:property name="color" value="0.8 0.8 0.8" />
-  <xacro:property name="opacity" value="1.0" />
-  <xacro:property name="mesh_ext" value="stl" />
-  <!-- Import all Gazebo-customization elements, including Gazebo colors -->
-  <xacro:include filename="$(find solo_description)/xacro/solo_control.xacro" />
-  <!-- This file is based on: https://atlas.is.localnet/confluence/display/AMDW/Quadruped+URDF+Files -->
-  <link name="base_link">
-    <!-- BASE LINK INERTIAL -->
-    <inertial>
-        <origin xyz="0 0 0" rpy="0 0 0" />
-        <mass value="1.16115091"/>
-        <!-- The base is extremely symmetrical. -->
-        <inertia ixx="0.00578574" ixy="0.0" ixz="0.0"
-                                  iyy="0.01938108" iyz="0.0"
-                                                   izz="0.02476124"
-        />
-    </inertial>
-    <!-- BASE LINK VISUAL -->
-    <visual>
-        <origin xyz="0 0 0" rpy="0 0 0" />
-        <geometry>
-          <mesh filename="file://$(find solo_description)/meshes/${mesh_ext}/solo12/solo_12_base.${mesh_ext}"/>
-        </geometry>
-        <material name="${color_name}">
-            <color rgba="${color} ${opacity}"/>
-        </material>
-    </visual>
-    <!-- BASE LINK COLLISION -->
-    <collision>
-        <origin xyz="0 0 0" rpy="0 0 0" />
-        <geometry>
-          <mesh filename="file://$(find solo_description)/meshes/${mesh_ext}/solo12/solo_12_base.${mesh_ext}"/>
-        </geometry>
-        <material name="${color_name}">
-            <color rgba="${color} ${opacity}"/>
-        </material>
-    </collision>
-    <!-- Bullet specific paramters -->
-    <contact>
-      <lateral_friction value="1.0"/>
-      <restitution value="0.5"/>
-    </contact>
-  </link> <!-- END BASE LINK -->
-  <!-- Include the legs -->
-  <xacro:include filename="leg.xacro"/>
-  <!-- Include the front left leg -->
-  <xacro:leg
-      prefix="FL"
-      is_front="true"
-      is_right="false"
-      has_side_motion="true"
-      mesh_ext="${mesh_ext}"
-      color_name="${color_name}"
-      color="${color}"
-      opacity="${opacity}"/>
-  <!-- Include the front right leg -->
-  <xacro:leg
-      prefix="FR"
-      is_front="true"
-      is_right="true"
-      has_side_motion="true"
-      mesh_ext="${mesh_ext}"
-      color_name="${color_name}"
-      color="${color}"
-      opacity="${opacity}"/>
-  <!-- Include the hind left leg -->
-  <xacro:leg
-      prefix="HL"
-      is_front="false"
-      is_right="false"
-      has_side_motion="true"
-      mesh_ext="${mesh_ext}"
-      color_name="${color_name}"
-      color="${color}"
-      opacity="${opacity}"/>
-  <!-- Include the hind right leg -->
-  <xacro:leg
-      prefix="HR"
-      is_front="false"
-      is_right="true"
-      has_side_motion="true"
-      mesh_ext="${mesh_ext}"
-      color_name="${color_name}"
-      color="${color}"
-      opacity="${opacity}"/>
+    xmlns:controller="http://playerstage.sourceforge.net/gazebo/xmlschema/#controller"
+    xmlns:interface="http://playerstage.sourceforge.net/gazebo/xmlschema/#interface"
+    xmlns:sensor="http://playerstage.sourceforge.net/gazebo/xmlschema/#sensor"
+    xmlns:xacro="http://playerstage.sourceforge.net/gazebo/xmlschema/#interface">
+    <xacro:property name="color_name" value="grey" />
+    <xacro:property name="color" value="0.8 0.8 0.8" />
+    <xacro:property name="opacity" value="1.0" />
+    <xacro:property name="mesh_ext" value="stl" />
+    <!-- Import all Gazebo-customization elements, including Gazebo colors -->
+    <xacro:include filename="$(find solo_description)/xacro/solo_gazebo.xacro" />
+    <!-- This file is based on: https://atlas.is.localnet/confluence/display/AMDW/Quadruped+URDF+Files -->
+    <link name="base_link">
+        <!-- BASE LINK INERTIAL -->
+        <inertial>
+            <origin xyz="0 0 0" rpy="0 0 0" />
+            <mass value="1.16115091"/>
+            <!-- The base is extremely symmetrical. -->
+            <inertia ixx="0.00578574" ixy="0.0"        ixz="0.0"
+                                      iyy="0.01938108" iyz="0.0"
+                                                       izz="0.02476124"
+            />
+        </inertial>
+        <!-- BASE LINK VISUAL -->
+        <visual>
+            <origin xyz="0 0 0" rpy="0 0 0" />
+            <geometry>
+                <mesh filename="file://$(find solo_description)/meshes/${mesh_ext}/solo12/solo_12_base.${mesh_ext}"/>
+            </geometry>
+            <material name="${color_name}">
+                <color rgba="${color} ${opacity}"/>
+            </material>
+        </visual>
+        <!-- BASE LINK COLLISION -->
+        <collision>
+            <origin xyz="0 0 0" rpy="0 0 0" />
+            <geometry>
+                <mesh filename="file://$(find solo_description)/meshes/${mesh_ext}/solo12/solo_12_base.${mesh_ext}"/>
+            </geometry>
+            <material name="${color_name}">
+                <color rgba="${color} ${opacity}"/>
+            </material>
+        </collision>
+        <!-- Bullet specific paramters -->
+        <contact>
+            <lateral_friction value="1.0"/>
+            <restitution value="0.5"/>
+        </contact>
+    </link> <!-- END BASE LINK -->
+    <!-- Include the legs -->
+    <xacro:include filename="leg.xacro"/>
+    <!-- Include the front left leg -->
+    <xacro:leg
+        prefix="FL"
+        is_front="true"
+        is_right="false"
+        has_side_motion="true"
+        mesh_ext="${mesh_ext}"
+        color_name="${color_name}"
+        color="${color}"
+        opacity="${opacity}"/>
+    <!-- Include the front right leg -->
+    <xacro:leg
+        prefix="FR"
+        is_front="true"
+        is_right="true"
+        has_side_motion="true"
+        mesh_ext="${mesh_ext}"
+        color_name="${color_name}"
+        color="${color}"
+        opacity="${opacity}"/>
+    <!-- Include the hind left leg -->
+    <xacro:leg
+        prefix="HL"
+        is_front="false"
+        is_right="false"
+        has_side_motion="true"
+        mesh_ext="${mesh_ext}"
+        color_name="${color_name}"
+        color="${color}"
+        opacity="${opacity}"/>
+    <!-- Include the hind right leg -->
+    <xacro:leg
+        prefix="HR"
+        is_front="false"
+        is_right="true"
+        has_side_motion="true"
+        mesh_ext="${mesh_ext}"
+        color_name="${color_name}"
+        color="${color}"
+        opacity="${opacity}"/>
 </robot>

File: xacro/solo8.urdf.xacro (robot description, xacro)
@@ -1,91 +1,91 @@
 <?xml version="1.0" ?>
 <robot name="solo"
-  xmlns:controller="http://playerstage.sourceforge.net/gazebo/xmlschema/#controller"
-  xmlns:interface="http://playerstage.sourceforge.net/gazebo/xmlschema/#interface"
-  xmlns:sensor="http://playerstage.sourceforge.net/gazebo/xmlschema/#sensor"
-  xmlns:xacro="http://playerstage.sourceforge.net/gazebo/xmlschema/#interface">
-  <xacro:property name="color_name" value="grey" />
-  <xacro:property name="color" value="0.8 0.8 0.8" />
-  <xacro:property name="opacity" value="1.0" />
-  <xacro:property name="mesh_ext" value="stl" />
-  <!-- This file is based on: https://atlas.is.localnet/confluence/display/AMDW/Quadruped+URDF+Files -->
-  <link name="base_link">
-    <!-- BASE LINK INERTIAL -->
-    <inertial>
-        <origin xyz="0 0 0" rpy="0 0 0" />
-        <mass value="1.43315091"/>
-        <!-- The base is extremely symmetrical. -->
-        <inertia ixx="0.00578574" ixy="0.0" ixz="0.0"
-                                  iyy="0.01938108" iyz="0.0"
-                                                   izz="0.02476124"
-        />
-    </inertial>
-    <!-- BASE LINK VISUAL -->
-    <visual>
-        <origin xyz="0 0 0" rpy="0 0 0" />
-        <geometry>
-          <mesh filename="file://$(find solo_description)/meshes/${mesh_ext}/with_foot/solo_body.${mesh_ext}"/>
-        </geometry>
-        <material name="${color_name}">
-            <color rgba="${color} ${opacity}"/>
-        </material>
-    </visual>
-    <!-- BASE LINK COLLISION -->
-    <collision>
-        <origin xyz="0 0 0" rpy="0 0 0" />
-        <geometry>
-          <mesh filename="file://$(find solo_description)/meshes/${mesh_ext}/with_foot/solo_body.${mesh_ext}"/>
-        </geometry>
-        <material name="${color_name}">
-            <color rgba="${color} ${opacity}"/>
-        </material>
-    </collision>
-    <!-- Bullet specific paramters -->
-    <contact>
-      <lateral_friction value="1.0"/>
-      <restitution value="0.5"/>
-    </contact>
-  </link> <!-- END BASE LINK -->
-  <!-- Include the legs -->
-  <xacro:include filename="leg.xacro"/>
-  <!-- Include the front left leg -->
-  <xacro:leg
-      prefix="FL"
-      is_front="true"
-      is_right="false"
-      has_side_motion="false"
-      mesh_ext="${mesh_ext}"
-      color_name="${color_name}"
-      color="${color}"
-      opacity="${opacity}"/>
-  <!-- Include the front right leg -->
-  <xacro:leg
-      prefix="FR"
-      is_front="true"
-      is_right="true"
-      has_side_motion="false"
-      mesh_ext="${mesh_ext}"
-      color_name="${color_name}"
-      color="${color}"
-      opacity="${opacity}"/>
-  <!-- Include the hind left leg -->
-  <xacro:leg
-      prefix="HL"
-      is_front="false"
-      is_right="false"
-      has_side_motion="false"
-      mesh_ext="${mesh_ext}"
-      color_name="${color_name}"
-      color="${color}"
-      opacity="${opacity}"/>
-  <!-- Include the hind right leg -->
-  <xacro:leg
-      prefix="HR"
-      is_front="false"
-      is_right="true"
-      has_side_motion="false"
-      mesh_ext="${mesh_ext}"
-      color_name="${color_name}"
-      color="${color}"
-      opacity="${opacity}"/>
+    xmlns:controller="http://playerstage.sourceforge.net/gazebo/xmlschema/#controller"
+    xmlns:interface="http://playerstage.sourceforge.net/gazebo/xmlschema/#interface"
+    xmlns:sensor="http://playerstage.sourceforge.net/gazebo/xmlschema/#sensor"
+    xmlns:xacro="http://playerstage.sourceforge.net/gazebo/xmlschema/#interface">
+    <xacro:property name="color_name" value="grey" />
+    <xacro:property name="color" value="0.8 0.8 0.8" />
+    <xacro:property name="opacity" value="1.0" />
+    <xacro:property name="mesh_ext" value="stl" />
+    <!-- This file is based on: https://atlas.is.localnet/confluence/display/AMDW/Quadruped+URDF+Files -->
+    <link name="base_link">
+        <!-- BASE LINK INERTIAL -->
+        <inertial>
+            <origin xyz="0 0 0" rpy="0 0 0" />
+            <mass value="1.43315091"/>
+            <!-- The base is extremely symmetrical. -->
+            <inertia ixx="0.00578574" ixy="0.0"        ixz="0.0"
+                                      iyy="0.01938108" iyz="0.0"
+                                                       izz="0.02476124"
+            />
+        </inertial>
+        <!-- BASE LINK VISUAL -->
+        <visual>
+            <origin xyz="0 0 0" rpy="0 0 0" />
+            <geometry>
+                <mesh filename="file://$(find solo_description)/meshes/${mesh_ext}/with_foot/solo_body.${mesh_ext}"/>
+            </geometry>
+            <material name="${color_name}">
+                <color rgba="${color} ${opacity}"/>
+            </material>
+        </visual>
+        <!-- BASE LINK COLLISION -->
+        <collision>
+            <origin xyz="0 0 0" rpy="0 0 0" />
+            <geometry>
+                <mesh filename="file://$(find solo_description)/meshes/${mesh_ext}/with_foot/solo_body.${mesh_ext}"/>
+            </geometry>
+            <material name="${color_name}">
+                <color rgba="${color} ${opacity}"/>
+            </material>
+        </collision>
+        <!-- Bullet specific paramters -->
+        <contact>
+            <lateral_friction value="1.0"/>
+            <restitution value="0.5"/>
+        </contact>
+    </link> <!-- END BASE LINK -->
+    <!-- Include the legs -->
+    <xacro:include filename="leg.xacro"/>
+    <!-- Include the front left leg -->
+    <xacro:leg
+        prefix="FL"
+        is_front="true"
+        is_right="false"
+        has_side_motion="false"
+        mesh_ext="${mesh_ext}"
+        color_name="${color_name}"
+        color="${color}"
+        opacity="${opacity}"/>
+    <!-- Include the front right leg -->
+    <xacro:leg
+        prefix="FR"
+        is_front="true"
+        is_right="true"
+        has_side_motion="false"
+        mesh_ext="${mesh_ext}"
+        color_name="${color_name}"
+        color="${color}"
+        opacity="${opacity}"/>
+    <!-- Include the hind left leg -->
+    <xacro:leg
+        prefix="HL"
+        is_front="false"
+        is_right="false"
+        has_side_motion="false"
+        mesh_ext="${mesh_ext}"
+        color_name="${color_name}"
+        color="${color}"
+        opacity="${opacity}"/>
+    <!-- Include the hind right leg -->
+    <xacro:leg
+        prefix="HR"
+        is_front="false"
+        is_right="true"
+        has_side_motion="false"
+        mesh_ext="${mesh_ext}"
+        color_name="${color_name}"
+        color="${color}"
+        opacity="${opacity}"/>
 </robot>
