Commit message: Add argument to use ros 2 control in simulation or real robot

File: xacro/solo12.urdf.xacro (robot description, xacro)
@@ -11,4 +11,6 @@
     <xacro:arg name="remove_shank_collisions" default="False"/>
     <xacro:property name="remove_shank_collisions" default="$(arg remove_shank_collisions)"/>
+    <xacro:arg name="sim" default="False"/>
+    <xacro:property name="sim" default="$(arg sim)"/>
     <!-- Import all Gazebo-customization elements, including Gazebo colors -->
     <xacro:include filename="$(find solo_description)/xacro/solo12_gazebo.xacro" />

File: xacro/solo12_gazebo.xacro (robot description, xacro)
@@ -1,45 +1,47 @@
 <?xml version="1.0"?>
 <robot xmlns:xacro="http://www.ros.org/wiki/xacro">
-    <xacro:macro name="ros2_control_joint" params="joint_name">
-        <joint name="${joint_name}">
-            <command_interface name="effort">
-                <param name="min">-20</param>
-                <param name="max"> 20</param>
-            </command_interface>
-            <state_interface name="position"/>
-            <state_interface name="velocity"/>
-            <state_interface name="effort"/>
-        </joint>
-    </xacro:macro>
-    <!-- ros2_control plugin -->
-    <ros2_control name="GazeboSystem" type="system">
-        <hardware>
-            <plugin>gazebo_ros2_control/GazeboSystem</plugin>
-        </hardware>
-        <xacro:ros2_control_joint joint_name="FL_HAA"></xacro:ros2_control_joint>
-        <xacro:ros2_control_joint joint_name="FL_HFE"></xacro:ros2_control_joint>
-        <xacro:ros2_control_joint joint_name="FL_KFE"></xacro:ros2_control_joint>
-        <xacro:ros2_control_joint joint_name="FR_HAA"></xacro:ros2_control_joint>
-        <xacro:ros2_control_joint joint_name="FR_HFE"></xacro:ros2_control_joint>
-        <xacro:ros2_control_joint joint_name="FR_KFE"></xacro:ros2_control_joint>
-        <xacro:ros2_control_joint joint_name="HL_HAA"></xacro:ros2_control_joint>
-        <xacro:ros2_control_joint joint_name="HL_HFE"></xacro:ros2_control_joint>
-        <xacro:ros2_control_joint joint_name="HL_KFE"></xacro:ros2_control_joint>
-        <xacro:ros2_control_joint joint_name="HR_HAA"></xacro:ros2_control_joint>
-        <xacro:ros2_control_joint joint_name="HR_HFE"></xacro:ros2_control_joint>
-        <xacro:ros2_control_joint joint_name="HR_KFE"></xacro:ros2_control_joint>
-        <sensor name="imu_sensor">
-            <state_interface name="orientation.x"/>
-            <state_interface name="orientation.y"/>
-            <state_interface name="orientation.z"/>
-            <state_interface name="orientation.w"/>
-            <state_interface name="angular_velocity.x"/>
-            <state_interface name="angular_velocity.y"/>
-            <state_interface name="angular_velocity.z"/>
-            <state_interface name="linear_acceleration.x"/>
-            <state_interface name="linear_acceleration.y"/>
-            <state_interface name="linear_acceleration.z"/>
-        </sensor>
-    </ros2_control>
+    <xacro:if value="${sim}">
+        <xacro:macro name="ros2_control_joint" params="joint_name">
+            <joint name="${joint_name}">
+                <command_interface name="effort">
+                    <param name="min">-20</param>
+                    <param name="max"> 20</param>
+                </command_interface>
+                <state_interface name="position"/>
+                <state_interface name="velocity"/>
+                <state_interface name="effort"/>
+            </joint>
+        </xacro:macro>
+        <!-- ros2_control plugin -->
+        <ros2_control name="GazeboSystem" type="system">
+            <hardware>
+                <plugin>gazebo_ros2_control/GazeboSystem</plugin>
+            </hardware>
+            <xacro:ros2_control_joint joint_name="FL_HAA"></xacro:ros2_control_joint>
+            <xacro:ros2_control_joint joint_name="FL_HFE"></xacro:ros2_control_joint>
+            <xacro:ros2_control_joint joint_name="FL_KFE"></xacro:ros2_control_joint>
+            <xacro:ros2_control_joint joint_name="FR_HAA"></xacro:ros2_control_joint>
+            <xacro:ros2_control_joint joint_name="FR_HFE"></xacro:ros2_control_joint>
+            <xacro:ros2_control_joint joint_name="FR_KFE"></xacro:ros2_control_joint>
+            <xacro:ros2_control_joint joint_name="HL_HAA"></xacro:ros2_control_joint>
+            <xacro:ros2_control_joint joint_name="HL_HFE"></xacro:ros2_control_joint>
+            <xacro:ros2_control_joint joint_name="HL_KFE"></xacro:ros2_control_joint>
+            <xacro:ros2_control_joint joint_name="HR_HAA"></xacro:ros2_control_joint>
+            <xacro:ros2_control_joint joint_name="HR_HFE"></xacro:ros2_control_joint>
+            <xacro:ros2_control_joint joint_name="HR_KFE"></xacro:ros2_control_joint>
+            <sensor name="imu_sensor">
+                <state_interface name="orientation.x"/>
+                <state_interface name="orientation.y"/>
+                <state_interface name="orientation.z"/>
+                <state_interface name="orientation.w"/>
+                <state_interface name="angular_velocity.x"/>
+                <state_interface name="angular_velocity.y"/>
+                <state_interface name="angular_velocity.z"/>
+                <state_interface name="linear_acceleration.x"/>
+                <state_interface name="linear_acceleration.y"/>
+                <state_interface name="linear_acceleration.z"/>
+            </sensor>
+        </ros2_control>
+    </xacro:if>
     <!-- Effort_controller -->
     <!-- <gazebo>
@@ -48,4 +50,16 @@
         </plugin>
     </gazebo> -->
+    <xacro:unless value="${sim}">
+        <ros2_control name="SOLO12_WB_Interface" type="system">
+            <hardware>
+                <plugin>solo12_interface/SOLO12_WB_Interface</plugin>
+                <param name="timeout">100</param>
+                <param name="command_type">0</param>
+                <param name="Kp">10.0</param>
+                <param name="Kv">0.0</param>
+                <param name="I_saturation">10.0</param>
+            </hardware>
+        </ros2_control>
+    </xacro:unless>
     <!-- IMU sensor -->
     <gazebo reference="base_link">
