Commit message: Edited package.xml and CMakeLists.txt + added new parameters and modified others in the controller .yaml file + added torque limits in the .xacro of the leg

File: xacro/leg.xacro (robot description, xacro)
@@ -19,5 +19,5 @@
         <parent link="base_link"/>
         <child link="${prefix}_SHOULDER"/>
-        <limit effort="1000" lower="-10" upper="10" velocity="1000"/>
+        <limit effort="10" lower="-10" upper="10" velocity="10"/>
         <!-- joints rotates around the x-axis -->
         <axis xyz="1 0 0"/>
@@ -152,5 +152,5 @@
         <parent link="${prefix}_SHOULDER"/>
         <child link="${prefix}_UPPER_LEG"/>
-        <limit effort="1000" lower="-10" upper="10" velocity="1000"/>
+        <limit effort="10" lower="-10" upper="10" velocity="10"/>
         <!-- joints rotates around the y-axis -->
         <axis xyz="0 1 0"/>
@@ -171,5 +171,5 @@
         <parent link="base_link"/>
         <child link="${prefix}_UPPER_LEG"/>
-        <limit effort="1000" lower="-10" upper="10" velocity="1000"/>
+        <limit effort="10" lower="-10" upper="10" velocity="10"/>
         <!-- joints rotates around the y-axis -->
         <axis xyz="0 1 0"/>
@@ -257,5 +257,5 @@
       <parent link="${prefix}_UPPER_LEG"/>
       <child link="${prefix}_LOWER_LEG"/>
-      <limit effort="1000" lower="-10" upper="10" velocity="1000"/>
+      <limit effort="10" lower="-10" upper="10" velocity="10"/>
       <!-- joints rotates around the y-axis -->
       <axis xyz="0 1 0"/>
@@ -350,5 +350,5 @@
       </xacro:if>
       <!-- Limits (usefull?) -->
-      <limit effort="1000" lower="-10" upper="10" velocity="1000"/>
+      <limit effort="10" lower="-10" upper="10" velocity="10"/>
       <!-- pybullet simulation parameters -->
       <dynamics damping="0.0" friction="0.0"/>

Commit message: Added contact sensors to the four feet + reduced the friction coefficient of the feet to 1

File: xacro/leg.xacro (robot description, xacro)
@@ -391,6 +391,6 @@
     </link> <!-- END LOWER LEG LINK -->
     <gazebo reference="${prefix}_FOOT">
-      <mu1>2</mu1>
-      <mu2>2</mu2>
+      <mu1>1</mu1>
+      <mu2>1</mu2>
     </gazebo>
   </xacro:macro>

File: xacro/solo12_gazebo.xacro (robot description, xacro)
@@ -117,3 +117,77 @@
         </sensor>
     </gazebo>
+    <!-- Contact sensors for the four feet -->
+    <!-- LF_FOOT -->
+    <gazebo reference="FL_LOWER_LEG">
+        <sensor name="LF_FOOT_contct_sensor" type="contact">
+            <always_on>true</always_on>
+            <update_rate>25.0</update_rate>
+            <contact>
+                <!-- gz sdf -p turtlebot3_burger.urdf.xacro and look for the name of the desired collision element. -->
+                <collision>FL_LOWER_LEG_fixed_joint_lump__FL_FOOT_collision_1</collision>
+                <!-- <collision>FL_LOWER_LEG_collision</collision> -->
+            </contact>
+            <plugin name="LF_FOOT_bumper" filename="libgazebo_ros_bumper.so">
+                <ros>
+                    <!-- <namespace>demo</namespace> -->
+                    <remapping>bumper_states:=/contact_force_sensors/LF</remapping>
+                </ros>
+                <frame_name>world</frame_name>
+            </plugin>
+        </sensor>
+    </gazebo>
+    <!-- RF_FOOT -->
+    <gazebo reference="FR_LOWER_LEG">
+        <sensor name="RF_FOOT_contct_sensor" type="contact">
+            <always_on>true</always_on>
+            <update_rate>25.0</update_rate>
+            <contact>
+                <!-- gz sdf -p turtlebot3_burger.urdf.xacro and look for the name of the desired collision element. -->
+                <collision>FR_LOWER_LEG_fixed_joint_lump__FR_FOOT_collision_1</collision>
+            </contact>
+            <plugin name="RF_FOOT_bumper" filename="libgazebo_ros_bumper.so">
+                <ros>
+                    <!-- <namespace>demo</namespace> -->
+                    <remapping>bumper_states:=/contact_force_sensors/RF</remapping>
+                </ros>
+                <frame_name>world</frame_name>
+            </plugin>
+        </sensor>
+    </gazebo>
+    <!-- LH_FOOT -->
+    <gazebo reference="HL_LOWER_LEG">
+        <sensor name="LH_FOOT_contct_sensor" type="contact">
+            <always_on>true</always_on>
+            <update_rate>25.0</update_rate>
+            <contact>
+                <!-- gz sdf -p turtlebot3_burger.urdf.xacro and look for the name of the desired collision element. -->
+                <collision>HL_LOWER_LEG_fixed_joint_lump__HL_FOOT_collision_1</collision>
+            </contact>
+            <plugin name="LH_FOOT_bumper" filename="libgazebo_ros_bumper.so">
+                <ros>
+                    <!-- <namespace>demo</namespace> -->
+                    <remapping>bumper_states:=/contact_force_sensors/LH</remapping>
+                </ros>
+                <frame_name>world</frame_name>
+            </plugin>
+        </sensor>
+    </gazebo>
+    <!-- RH_FOOT -->
+    <gazebo reference="HR_LOWER_LEG">
+        <sensor name="RH_FOOT_contct_sensor" type="contact">
+            <always_on>true</always_on>
+            <update_rate>25.0</update_rate>
+            <contact>
+                <!-- gz sdf -p turtlebot3_burger.urdf.xacro and look for the name of the desired collision element. -->
+                <collision>HR_LOWER_LEG_fixed_joint_lump__HR_FOOT_collision_1</collision>
+            </contact>
+            <plugin name="RH_FOOT_bumper" filename="libgazebo_ros_bumper.so">
+                <ros>
+                    <!-- <namespace>demo</namespace> -->
+                    <remapping>bumper_states:=/contact_force_sensors/RH</remapping>
+                </ros>
+                <frame_name>world</frame_name>
+            </plugin>
+        </sensor>
+    </gazebo>
 </robot>

Commit message: Added arg to remove the shank collisions

File: xacro/leg.xacro (robot description, xacro)
@@ -318,18 +318,20 @@
       </visual>
       <!-- LOWER LEG LINK COLLISION -->
-      <collision>
-        <origin xyz="0 0 0" rpy="0 0 0" />
-        <geometry>
-          <xacro:unless value="${is_right}">
-            <mesh filename="file://$(find solo_description)/meshes/${mesh_ext}/with_foot/solo_lower_leg_left_side.${mesh_ext}"/>
-          </xacro:unless>
-          <xacro:if value="${is_right}">
-            <mesh filename="file://$(find solo_description)/meshes/${mesh_ext}/with_foot/solo_lower_leg_right_side.${mesh_ext}"/>
-          </xacro:if>
-        </geometry>
-        <material name="${color_name}">
-            <color rgba="${color} ${opacity}"/>
-        </material>
-      </collision>
+      <xacro:unless value="${remove_shank_collisions}">
+        <collision>
+          <xacro:unless value="${is_right}">
+            <origin xyz="0  0.0075 -0.075" rpy="0 0 0" />
+          </xacro:unless>
+          <xacro:if value="${is_right}">
+            <origin xyz="0 -0.0075 -0.075" rpy="0 0 0" />
+          </xacro:if>
+          <geometry>
+            <box size="0.015 0.01 0.15"/>
+          </geometry>
+          <material name="${color_name}">
+              <color rgba="${color} ${opacity}"/>
+          </material>
+        </collision>
+      </xacro:unless>
       <!-- Bullet specific paramters -->
       <contact>
@@ -376,7 +378,7 @@
       <!-- FOOT COLLISION -->
       <collision>
-        <origin xyz="0 0 0" rpy="0 0 0" />
-        <geometry>
-            <mesh filename="file://$(find solo_description)/meshes/${mesh_ext}/with_foot/solo_foot.${mesh_ext}"/>
+        <origin xyz="0 0 0" rpy="1.57079632679 0 0" />
+        <geometry>
+          <sphere radius="0.015"/>
         </geometry>
         <material name="${color_name}">

File: xacro/solo12.urdf.xacro (robot description, xacro)
@@ -9,4 +9,6 @@
     <xacro:property name="opacity" value="1.0" />
     <xacro:property name="mesh_ext" value="stl" />
+    <xacro:arg name="remove_shank_collisions" default="False"/>
+    <xacro:property name="remove_shank_collisions" default="$(arg remove_shank_collisions)"/>
     <!-- Import all Gazebo-customization elements, including Gazebo colors -->
     <xacro:include filename="$(find solo_description)/xacro/solo12_gazebo.xacro" />

File: xacro/solo12_gazebo.xacro (robot description, xacro)
@@ -125,6 +125,10 @@
             <contact>
                 <!-- gz sdf -p turtlebot3_burger.urdf.xacro and look for the name of the desired collision element. -->
-                <collision>FL_LOWER_LEG_fixed_joint_lump__FL_FOOT_collision_1</collision>
-                <!-- <collision>FL_LOWER_LEG_collision</collision> -->
+                <xacro:if value="${remove_shank_collisions}">
+                    <collision>FL_LOWER_LEG_fixed_joint_lump__FL_FOOT_collision</collision>
+                </xacro:if>
+                <xacro:unless value="${remove_shank_collisions}">
+                    <collision>FL_LOWER_LEG_fixed_joint_lump__FL_FOOT_collision_1</collision>
+                </xacro:unless>
             </contact>
             <plugin name="LF_FOOT_bumper" filename="libgazebo_ros_bumper.so">
@@ -144,5 +148,10 @@
             <contact>
                 <!-- gz sdf -p turtlebot3_burger.urdf.xacro and look for the name of the desired collision element. -->
-                <collision>FR_LOWER_LEG_fixed_joint_lump__FR_FOOT_collision_1</collision>
+                <xacro:if value="${remove_shank_collisions}">
+                    <collision>FR_LOWER_LEG_fixed_joint_lump__FR_FOOT_collision</collision>
+                </xacro:if>
+                <xacro:unless value="${remove_shank_collisions}">
+                    <collision>FR_LOWER_LEG_fixed_joint_lump__FR_FOOT_collision_1</collision>
+                </xacro:unless>
             </contact>
             <plugin name="RF_FOOT_bumper" filename="libgazebo_ros_bumper.so">
@@ -162,5 +171,10 @@
             <contact>
                 <!-- gz sdf -p turtlebot3_burger.urdf.xacro and look for the name of the desired collision element. -->
-                <collision>HL_LOWER_LEG_fixed_joint_lump__HL_FOOT_collision_1</collision>
+                <xacro:if value="${remove_shank_collisions}">
+                    <collision>HL_LOWER_LEG_fixed_joint_lump__HL_FOOT_collision</collision>
+                </xacro:if>
+                <xacro:unless value="${remove_shank_collisions}">
+                    <collision>HL_LOWER_LEG_fixed_joint_lump__HL_FOOT_collision_1</collision>
+                </xacro:unless>
             </contact>
             <plugin name="LH_FOOT_bumper" filename="libgazebo_ros_bumper.so">
@@ -180,5 +194,10 @@
             <contact>
                 <!-- gz sdf -p turtlebot3_burger.urdf.xacro and look for the name of the desired collision element. -->
-                <collision>HR_LOWER_LEG_fixed_joint_lump__HR_FOOT_collision_1</collision>
+                <xacro:if value="${remove_shank_collisions}">
+                    <collision>HR_LOWER_LEG_fixed_joint_lump__HR_FOOT_collision</collision>
+                </xacro:if>
+                <xacro:unless value="${remove_shank_collisions}">
+                    <collision>HR_LOWER_LEG_fixed_joint_lump__HR_FOOT_collision_1</collision>
+                </xacro:unless>
             </contact>
             <plugin name="RH_FOOT_bumper" filename="libgazebo_ros_bumper.so">
