Commit message: Removed comments to avoid Gazebo bug

File: xacro/leg.xacro (robot description, xacro)
@@ -1,6 +1,4 @@
 <?xml version="1.0"?>
 <robot xmlns:xacro="http://playerstage.sourceforge.net/gazebo/xmlschema/#interface" name="solo">
-  <!-- See TODO: add the wiki link here -->
-  <!-- These are absoulte distance value, the sign are decided below -->
   <xacro:property name="base_2_HAA_x" value="${194.60 * 0.001}" />
   <xacro:property name="base_2_HAA_y" value="${87.50 * 0.001}" />
@@ -12,5 +10,4 @@
   <xacro:property name="KFE_2_FOOT_y" value="${8.0 * 0.001}" />
   <xacro:property name="KFE_2_FOOT_z" value="${160.00 * 0.001}" />
-  <!-- Macro defining solo leg. -->
   <xacro:macro name="leg" params="prefix is_front is_right has_side_motion
                                   mesh_ext color_name color opacity">
@@ -20,7 +17,5 @@
         <child link="${prefix}_SHOULDER"/>
         <limit effort="10" lower="-10" upper="10" velocity="10"/>
-        <!-- joints rotates around the x-axis -->
         <axis xyz="1 0 0"/>
-        <!-- placement of the joint -->
         <xacro:if value="${is_front}">
           <xacro:unless value="${is_right}">
@@ -39,11 +34,7 @@
           </xacro:if>
         </xacro:unless>
-        <!-- pybullet simulation parameters -->
         <dynamics damping="0.0" friction="0.0"/>
       </joint>
       <link name="${prefix}_SHOULDER">
-        <!-- TODO: Update inertias. -->
-        <!-- create a dummy shoulder link to join the two joints -->
-        <!-- HAA VISUAL -->
         <visual>
             <xacro:unless value="${is_right}">
@@ -79,5 +70,4 @@
             </material>
         </visual>
-        <!-- HAA LINK COLLISION -->
         <collision>
                 <xacro:unless value="${is_right}">
@@ -117,5 +107,4 @@
           <xacro:if value="${is_front}">
             <xacro:unless value="${is_right}">
-              <!-- HAA body inertia -->
               <origin xyz="-0.07870700 0.01 0." rpy="0 0 0" />
               <inertia ixx="0.00003024" ixy="0.00004671" ixz="0.0"
@@ -124,5 +113,4 @@
             </xacro:unless>
             <xacro:if value="${is_right}">
-              <!-- HAA body inertia -->
               <origin xyz="-0.07870700 -0.01 0." rpy="0 0 0" />
               <inertia ixx="0.00003024" ixy="-0.00004671" ixz="0.0"
@@ -133,5 +121,4 @@
           <xacro:unless value="${is_front}">
             <xacro:unless value="${is_right}">
-              <!-- HAA body inertia -->
               <origin xyz="0.07870700 0.01 0." rpy="0 0 0" />
               <inertia ixx="0.00003024" ixy="0.00004671" ixz="0.0"
@@ -140,5 +127,4 @@
             </xacro:unless>
             <xacro:if value="${is_right}">
-              <!-- HAA body inertia -->
               <origin xyz="0.07870700 -0.01 0." rpy="0 0 0" />
               <inertia ixx="0.00003024" ixy="-0.00004671" ixz="0.0"
@@ -153,7 +139,5 @@
         <child link="${prefix}_UPPER_LEG"/>
         <limit effort="10" lower="-10" upper="10" velocity="10"/>
-        <!-- joints rotates around the y-axis -->
         <axis xyz="0 1 0"/>
-        <!-- placement of the joint -->
         <xacro:if value="${is_right}">
           <origin xyz="0 ${-HAA_2_HFE_y} 0" rpy="0 0 0" />
@@ -162,17 +146,13 @@
           <origin xyz="0 ${HAA_2_HFE_y} 0" rpy="0 0 0" />
         </xacro:unless>
-        <!-- pybullet simulation parameters -->
         <dynamics damping="0.0" friction="0.0"/>
       </joint>
     </xacro:if>
     <xacro:unless value="${has_side_motion}">
-      <!-- Joint between the base and the ${prefix} upper leg -->
       <joint name="${prefix}_HFE" type="revolute">
         <parent link="base_link"/>
         <child link="${prefix}_UPPER_LEG"/>
         <limit effort="10" lower="-10" upper="10" velocity="10"/>
-        <!-- joints rotates around the y-axis -->
         <axis xyz="0 1 0"/>
-        <!-- placement of the joint -->
         <xacro:if value="${is_front}">
           <xacro:unless value="${is_right}">
@@ -191,12 +171,9 @@
           </xacro:if>
         </xacro:unless>
-        <!-- pybullet simulation parameters -->
         <dynamics damping="0.0" friction="0.0"/>
       </joint>
     </xacro:unless>
     <link name="${prefix}_UPPER_LEG">
-      <!-- UPPER LEG LINK INERTIAL -->
       <xacro:unless value="${is_right}">
-        <!-- Left upper leg inertia -->
         <inertial>
         <origin xyz="0.00001377 0.01935853 -0.07870700" rpy="0 0 0" />
@@ -208,5 +185,4 @@
       </xacro:unless>
       <xacro:if value="${is_right}">
-        <!-- Right upper leg inertia -->
         <inertial>
         <origin xyz="-0.00001377 -0.01935853 -0.07870700" rpy="0 0 0" />
@@ -217,5 +193,4 @@
         </inertial>
       </xacro:if>
-      <!-- UPPER LEG LINK VISUAL -->
       <visual>
         <origin xyz="0 0 0" rpy="0 0 0" />
@@ -232,5 +207,4 @@
         </material>
       </visual>
-      <!-- UPPER LEG LINK COLLISION -->
       <collision>
         <origin xyz="0 0 0" rpy="0 0 0" />
@@ -247,18 +221,14 @@
         </material>
       </collision>
-      <!-- Bullet specific paramters -->
       <contact>
         <lateral_friction value="1.0"/>
         <restitution value="0.5"/>
       </contact>
-    </link> <!-- END UPPER LEG LINK -->
-    <!-- KFE: Joint between the upper leg and the lower leg -->
+    </link>
     <joint name="${prefix}_KFE" type="revolute">
       <parent link="${prefix}_UPPER_LEG"/>
       <child link="${prefix}_LOWER_LEG"/>
       <limit effort="10" lower="-10" upper="10" velocity="10"/>
-      <!-- joints rotates around the y-axis -->
       <axis xyz="0 1 0"/>
-      <!-- placement of the joint -->
       <xacro:if value="${is_front}">
         <xacro:unless value="${is_right}">
@@ -277,11 +247,8 @@
         </xacro:if>
       </xacro:unless>
-      <!-- pybullet simulation parameters -->
       <dynamics damping="0.0" friction="0.0"/>
     </joint>
     <link name="${prefix}_LOWER_LEG">
-      <!-- LOWER LEG LINK INERTIAL -->
       <xacro:unless value="${is_right}">
-        <!-- Left lower leg inertia -->
         <inertial>
         <origin xyz="0.0 0.00787644 -0.08928215" rpy="0 0 0" />
@@ -293,5 +260,4 @@
       </xacro:unless>
       <xacro:if value="${is_right}">
-        <!-- Right lower leg inertia -->
         <inertial>
         <origin xyz="0.0 0.00787644 -0.08928215" rpy="0 0 0" />
@@ -302,5 +268,4 @@
         </inertial>
       </xacro:if>
-      <!-- LOWER LEG LINK VISUAL -->
       <visual>
         <origin xyz="0 0 0" rpy="0 0 0" />
@@ -317,5 +282,4 @@
         </material>
       </visual>
-      <!-- LOWER LEG LINK COLLISION -->
       <xacro:unless value="${remove_shank_collisions}">
         <collision>
@@ -334,15 +298,12 @@
         </collision>
       </xacro:unless>
-      <!-- Bullet specific paramters -->
       <contact>
         <lateral_friction value="1.0"/>
         <restitution value="0.5"/>
       </contact>
-    </link> <!-- END LOWER LEG LINK -->
-    <!-- KFE: Joint between the upper leg and the lower leg -->
+    </link>
     <joint name="${prefix}_ANKLE" type="fixed">
       <parent link="${prefix}_LOWER_LEG"/>
       <child link="${prefix}_FOOT"/>
-      <!-- Joint placement -->
       <xacro:unless value="${is_right}">
         <origin xyz="0 ${KFE_2_FOOT_y} ${-KFE_2_FOOT_z}" rpy="0 0 0" />
@@ -351,12 +312,8 @@
         <origin xyz="0 ${-KFE_2_FOOT_y} ${-KFE_2_FOOT_z}" rpy="0 0 0" />
       </xacro:if>
-      <!-- Limits (usefull?) -->
       <limit effort="10" lower="-10" upper="10" velocity="10"/>
-      <!-- pybullet simulation parameters -->
       <dynamics damping="0.0" friction="0.0"/>
     </joint>
     <link name="${prefix}_FOOT">
-      <!-- FOOT INERTIAL -->
-      <!-- This link is symmetrical left or right -->
       <inertial>
         <origin xyz="0 0 0.00035767" rpy="0 0 0" />
@@ -366,5 +323,4 @@
                                                     izz="0.00000053"/>
      </inertial>
-      <!-- FOOT VISUAL -->
       <visual>
         <origin xyz="0 0 0" rpy="0 0 0" />
@@ -376,5 +332,4 @@
         </material>
       </visual>
-      <!-- FOOT COLLISION -->
       <collision>
         <origin xyz="0 0 0" rpy="1.57079632679 0 0" />
@@ -386,10 +341,9 @@
         </material>
       </collision>
-      <!-- Bullet specific paramters -->
       <contact>
         <lateral_friction value="1.0"/>
         <restitution value="0.5"/>
       </contact>
-    </link> <!-- END LOWER LEG LINK -->
+    </link>
     <gazebo reference="${prefix}_FOOT">
       <mu1>1</mu1>

File: xacro/solo12.urdf.xacro (robot description, xacro)
@@ -11,15 +11,11 @@
     <xacro:arg name="remove_shank_collisions" default="False"/>
     <xacro:property name="remove_shank_collisions" default="$(arg remove_shank_collisions)"/>
-    <xacro:arg name="sim" default="False"/>
+    <xacro:arg name="sim" default="True"/>
     <xacro:property name="sim" default="$(arg sim)"/>
-    <!-- Import all Gazebo-customization elements, including Gazebo colors -->
     <xacro:include filename="$(find solo_description)/xacro/solo12_gazebo.xacro" />
-    <!-- This file is based on: https://atlas.is.localnet/confluence/display/AMDW/Quadruped+URDF+Files -->
     <link name="base_link">
-        <!-- BASE LINK INERTIAL -->
         <inertial>
             <origin xyz="0 0 0" rpy="0 0 0" />
             <mass value="1.16115091"/>
-            <!-- The base is extremely symmetrical. -->
             <inertia ixx="0.00578574" ixy="0.0"        ixz="0.0"
                                       iyy="0.01938108" iyz="0.0"
@@ -27,5 +23,4 @@
             />
         </inertial>
-        <!-- BASE LINK VISUAL -->
         <visual>
             <origin xyz="0 0 0" rpy="0 0 0" />
@@ -37,5 +32,4 @@
             </material>
         </visual>
-        <!-- BASE LINK COLLISION -->
         <collision>
             <origin xyz="0 0 0" rpy="0 0 0" />
@@ -47,13 +41,10 @@
             </material>
         </collision>
-        <!-- Bullet specific paramters -->
         <contact>
             <lateral_friction value="1.0"/>
             <restitution value="0.5"/>
         </contact>
-    </link> <!-- END BASE LINK -->
-    <!-- Include the legs -->
+    </link>
     <xacro:include filename="leg.xacro"/>
-    <!-- Include the front left leg -->
     <xacro:leg
         prefix="FL"
@@ -65,5 +56,4 @@
         color="${color}"
         opacity="${opacity}"/>
-    <!-- Include the front right leg -->
     <xacro:leg
         prefix="FR"
@@ -75,5 +65,4 @@
         color="${color}"
         opacity="${opacity}"/>
-    <!-- Include the hind left leg -->
     <xacro:leg
         prefix="HL"
@@ -85,5 +74,4 @@
         color="${color}"
         opacity="${opacity}"/>
-    <!-- Include the hind right leg -->
     <xacro:leg
         prefix="HR"

File: xacro/solo12_gazebo.xacro (robot description, xacro)
@@ -13,5 +13,4 @@
             </joint>
         </xacro:macro>
-        <!-- ros2_control plugin -->
         <ros2_control name="GazeboSystem" type="system">
             <hardware>
@@ -43,11 +42,10 @@
             </sensor>
         </ros2_control>
+        <gazebo>
+            <plugin filename="libgazebo_ros2_control.so" name="gazebo_ros2_control">
+                <parameters>$(find robot_control)/config/gazebo/solo12_controller_effort.yaml</parameters>
+            </plugin>
+        </gazebo>
     </xacro:if>
-    <!-- Effort_controller -->
-    <!-- <gazebo>
-        <plugin filename="libgazebo_ros2_control.so" name="gazebo_ros2_control">
-            <parameters>$(find robot_control)/config/gazebo/solo12_controller_effort.yaml</parameters>
-        </plugin>
-    </gazebo> -->
     <xacro:unless value="${sim}">
         <ros2_control name="SOLO12_WB_Interface" type="system">
@@ -62,17 +60,8 @@
         </ros2_control>
     </xacro:unless>
-    <!-- IMU sensor -->
     <gazebo reference="base_link">
         <sensor name="imu_sensor" type="imu">
             <always_on>true</always_on>
             <update_rate>400</update_rate>
-            <!-- <plugin name="imu_plugin" filename="libgazebo_ros_imu_sensor.so">
-                <ros>
-                    <namespace>/imu</namespace>
-                    <remapping>~/out:=data</remapping>
-                </ros>
-                <frame_name>base</frame_name>
-                <initial_orientation_as_reference>false</initial_orientation_as_reference>
-            </plugin> -->
             <imu>
                 <angular_velocity>
@@ -80,7 +69,4 @@
                         <noise type="gaussian">
                         <mean>0.0</mean>
-                            <!-- <stddev>2e-4</stddev>
-                            <bias_mean>0.0000075</bias_mean>
-                            <bias_stddev>0.0000008</bias_stddev> -->
                             <stddev>0.0</stddev>
                             <bias_mean>0.00000</bias_mean>
@@ -91,7 +77,4 @@
                         <noise type="gaussian">
                         <mean>0.0</mean>
-                            <!-- <stddev>2e-4</stddev>
-                            <bias_mean>0.0000075</bias_mean>
-                            <bias_stddev>0.0000008</bias_stddev> -->
                             <stddev>0.0</stddev>
                             <bias_mean>0.00000</bias_mean>
@@ -102,7 +85,4 @@
                         <noise type="gaussian">
                         <mean>0.0</mean>
-                            <!-- <stddev>2e-4</stddev>
-                            <bias_mean>0.0000075</bias_mean>
-                            <bias_stddev>0.0000008</bias_stddev> -->
                             <stddev>0.0</stddev>
                             <bias_mean>0.00000</bias_mean>
@@ -115,7 +95,4 @@
                         <noise type="gaussian">
                             <mean>0.0</mean>
-                            <!-- <stddev>1.7e-2</stddev>
-                            <bias_mean>0.1</bias_mean>
-                            <bias_stddev>0.001</bias_stddev> -->
                             <stddev>0.0</stddev>
                             <bias_mean>0.0</bias_mean>
@@ -126,7 +103,4 @@
                         <noise type="gaussian">
                             <mean>0.0</mean>
-                            <!-- <stddev>1.7e-2</stddev>
-                            <bias_mean>0.1</bias_mean>
-                            <bias_stddev>0.001</bias_stddev> -->
                             <stddev>0.0</stddev>
                             <bias_mean>0.0</bias_mean>
@@ -137,7 +111,4 @@
                         <noise type="gaussian">
                             <mean>0.0</mean>
-                            <!-- <stddev>1.7e-2</stddev>
-                            <bias_mean>0.1</bias_mean>
-                            <bias_stddev>0.001</bias_stddev> -->
                             <stddev>0.0</stddev>
                             <bias_mean>0.0</bias_mean>
@@ -149,6 +120,4 @@
         </sensor>
     </gazebo>
-    <!-- Contact sensors for the four feet -->
-    <!-- LF_FOOT -->
     <gazebo reference="FL_LOWER_LEG">
         <sensor name="LF_FOOT_contct_sensor" type="contact">
@@ -156,5 +125,4 @@
             <update_rate>25.0</update_rate>
             <contact>
-                <!-- gz sdf -p turtlebot3_burger.urdf.xacro and look for the name of the desired collision element. -->
                 <xacro:if value="${remove_shank_collisions}">
                     <collision>FL_LOWER_LEG_fixed_joint_lump__FL_FOOT_collision</collision>
@@ -166,5 +134,4 @@
             <plugin name="LF_FOOT_bumper" filename="libgazebo_ros_bumper.so">
                 <ros>
-                    <!-- <namespace>demo</namespace> -->
                     <remapping>bumper_states:=/contact_force_sensors/LF</remapping>
                 </ros>
@@ -173,5 +140,4 @@
         </sensor>
     </gazebo>
-    <!-- RF_FOOT -->
     <gazebo reference="FR_LOWER_LEG">
         <sensor name="RF_FOOT_contct_sensor" type="contact">
@@ -179,5 +145,4 @@
             <update_rate>25.0</update_rate>
             <contact>
-                <!-- gz sdf -p turtlebot3_burger.urdf.xacro and look for the name of the desired collision element. -->
                 <xacro:if value="${remove_shank_collisions}">
                     <collision>FR_LOWER_LEG_fixed_joint_lump__FR_FOOT_collision</collision>
@@ -189,5 +154,4 @@
             <plugin name="RF_FOOT_bumper" filename="libgazebo_ros_bumper.so">
                 <ros>
-                    <!-- <namespace>demo</namespace> -->
                     <remapping>bumper_states:=/contact_force_sensors/RF</remapping>
                 </ros>
@@ -196,5 +160,4 @@
         </sensor>
     </gazebo>
-    <!-- LH_FOOT -->
     <gazebo reference="HL_LOWER_LEG">
         <sensor name="LH_FOOT_contct_sensor" type="contact">
@@ -202,5 +165,4 @@
             <update_rate>25.0</update_rate>
             <contact>
-                <!-- gz sdf -p turtlebot3_burger.urdf.xacro and look for the name of the desired collision element. -->
                 <xacro:if value="${remove_shank_collisions}">
                     <collision>HL_LOWER_LEG_fixed_joint_lump__HL_FOOT_collision</collision>
@@ -212,5 +174,4 @@
             <plugin name="LH_FOOT_bumper" filename="libgazebo_ros_bumper.so">
                 <ros>
-                    <!-- <namespace>demo</namespace> -->
                     <remapping>bumper_states:=/contact_force_sensors/LH</remapping>
                 </ros>
@@ -219,5 +180,4 @@
         </sensor>
     </gazebo>
-    <!-- RH_FOOT -->
     <gazebo reference="HR_LOWER_LEG">
         <sensor name="RH_FOOT_contct_sensor" type="contact">
@@ -225,5 +185,4 @@
             <update_rate>25.0</update_rate>
             <contact>
-                <!-- gz sdf -p turtlebot3_burger.urdf.xacro and look for the name of the desired collision element. -->
                 <xacro:if value="${remove_shank_collisions}">
                     <collision>HR_LOWER_LEG_fixed_joint_lump__HR_FOOT_collision</collision>
@@ -235,5 +194,4 @@
             <plugin name="RH_FOOT_bumper" filename="libgazebo_ros_bumper.so">
                 <ros>
-                    <!-- <namespace>demo</namespace> -->
                     <remapping>bumper_states:=/contact_force_sensors/RH</remapping>
                 </ros>
